Commit message: Update nico_base.urdf.xacro
collision sensor cylinder fixed

File: ros-rl-env/catkin_ws/src/hector_quadrotor_noetic/hector_quadrotor/hector_quadrotor_description/urdf/nico_base.urdf.xacro (robot description, xacro)
@@ -40,5 +40,5 @@
         <origin xyz="0 0 -0.1" rpy="0 0 0" />
         <geometry>
-          <cylinder length="0.35" radius="0.4"/>
+          <cylinder length="0.40" radius="0.4"/>
         </geometry>
         <material name="ChassisRed">
@@ -49,5 +49,5 @@
         <origin xyz="0 0 0" rpy="0 0 0"/>
         <geometry>
-          <cylinder length="0.01" radius="0.4"/>
+          <cylinder length="0.40" radius="0.4"/>
         </geometry>
       </collision>

Commit message: Update nico_base.urdf.xacro
collisioon sensor cylinder modified

File: ros-rl-env/catkin_ws/src/hector_quadrotor_noetic/hector_quadrotor/hector_quadrotor_description/urdf/nico_base.urdf.xacro (robot description, xacro)
@@ -47,5 +47,5 @@
       </visual>
       <collision>
-        <origin xyz="0 0 0" rpy="0 0 0"/>
+        <origin xyz="0 0 -0.1" rpy="0 0 0"/>
         <geometry>
           <cylinder length="0.40" radius="0.4"/>
